Commit message: minor edits

File: iauv_description/urdf/g1000_bravo.urdf.xacro (robot description, xacro)
@@ -2,5 +2,5 @@
 <robot name="girona1000" xmlns:xacro="http://www.ros.org/wiki/xacro">
   <xacro:arg name="robot_namespace" default="girona1000"/>
-  <xacro:arg name="bravo_right_namespace" default="$(arg robot_namespace)/bravo_right"/>
+  <xacro:arg name="bravo_namespace" default="$(arg robot_namespace)/bravo"/>
   <!-- Include Girona1000 -->
   <xacro:include filename="$(find girona1000_description)/urdf/girona1000_intervention.urdf.xacro"/>
@@ -20,12 +20,12 @@
     filename="$(find blueprintlab_reachbravo7_manipulator_description)/urdf/end_effectors/jaws_macro.urdf.xacro"/>
   <!-- Add manipulators-->
-  <xacro:reach_bravo7 prefix="$(arg bravo_right_namespace)" link6_lowlimit="0.0" link6_uplimit="3.14"/>
+  <xacro:reach_bravo7 prefix="$(arg bravo_namespace)" link6_lowlimit="0.0" link6_uplimit="3.14"/>
   <!-- Attach manipulator to base -->
-  <joint name="girona1000_to_bravo_right" type="fixed">
+  <joint name="girona1000_to_bravo" type="fixed">
     <parent link="$(arg robot_namespace)/origin"/>
-    <child link="$(arg bravo_right_namespace)/base_link"/>
+    <child link="$(arg bravo_namespace)/base_link"/>
     <origin rpy="${pi} 0.0 0.175" xyz="0.7322 0.1382 0.485"/>
   </joint>
-  <xacro:reach_bravo7_jaws prefix="$(arg bravo_right_namespace)"/>
+  <xacro:reach_bravo7_jaws prefix="$(arg bravo_namespace)"/>
   <link name="$(arg robot_namespace)/depth_cam_link"/>
   <joint name="$(arg robot_namespace)/depth_cam_joint" type="fixed">
@@ -34,8 +34,8 @@
     <origin rpy="1.309 0 1.57" xyz="0.7322 -0.1382 0.485"/>
   </joint>
-  <link name="$(arg bravo_right_namespace)/gripper_camera"/>
+  <link name="$(arg bravo_namespace)/gripper_camera"/>
   <joint name="camera_joint" type="fixed">
-    <parent link="$(arg bravo_right_namespace)/jaws_base_link"/>
-    <child link="$(arg bravo_right_namespace)/gripper_camera"/>
+    <parent link="$(arg bravo_namespace)/jaws_base_link"/>
+    <child link="$(arg bravo_namespace)/gripper_camera"/>
     <origin rpy="0 0 0" xyz="0 0 0.05"/>
   </joint>

Commit message: added luma tfs

File: iauv_description/urdf/g1000_bravo.urdf.xacro (robot description, xacro)
@@ -40,3 +40,9 @@
     <origin rpy="0 0 0" xyz="0 0 0.05"/>
   </joint>
+  <link name="$(arg robot_namespace)/luma_link"/>
+  <joint name="luma_joint" type="fixed">
+    <parent link="$(arg robot_namespace)/origin"/>
+    <child link="$(arg robot_namespace)/luma_link"/>
+    <origin rpy="0 -1.57 0" xyz="-0.5 0 0.3"/>
+  </joint>
 </robot>

Commit message: debranding device

File: iauv_description/urdf/g1000_bravo.urdf.xacro (robot description, xacro)
@@ -40,8 +40,8 @@
     <origin rpy="0 0 0" xyz="0 0 0.05"/>
   </joint>
-  <link name="$(arg robot_namespace)/luma_link"/>
-  <joint name="luma_joint" type="fixed">
+  <link name="$(arg robot_namespace)/vlc_link"/>
+  <joint name="vlc_joint" type="fixed">
     <parent link="$(arg robot_namespace)/origin"/>
-    <child link="$(arg robot_namespace)/luma_link"/>
+    <child link="$(arg robot_namespace)/vlc_link"/>
     <origin rpy="0 -1.57 0" xyz="-0.5 0 0.3"/>
   </joint>

Commit message: including self collisions

File: iauv_description/urdf/g1000_bravo.urdf.xacro (robot description, xacro)
@@ -46,3 +46,18 @@
     <origin rpy="0 -1.57 0" xyz="-0.5 0 0.3"/>
   </joint>
+  <xacro:property name="x_col" value="0.7322"/>
+  <xacro:property name="z_col" value="0.485"/>
+  <link name="$(arg robot_namespace)/collision">
+    <collision>
+      <geometry>
+        <box size="1.0 0.1 1.0"/>
+      </geometry>
+      <origin rpy="0.0 0.0 0.0" xyz="-0.1 0.0 0.0"/>
+    </collision>
+  </link>
+  <joint name="collision_joint" type="fixed">
+    <parent link="$(arg robot_namespace)/origin"/>
+    <child link="$(arg robot_namespace)/collision"/>
+    <origin rpy="0.0 0.0 0.0" xyz="${x_col} 0.0 ${z_col}"/>
+  </joint>
 </robot>

Commit message: arm in conditional now

File: iauv_description/urdf/g1000_bravo.urdf.xacro (robot description, xacro)
@@ -13,19 +13,21 @@
     <origin rpy="${pi/2} 0.0 ${pi/2}" xyz="0.7322 -0.1382 0.385"/>
   </joint>
-  <!-- Include manipulators -->
-  <xacro:include
-    filename="$(find blueprintlab_reachbravo7_manipulator_description)/urdf/bravo7_macro.urdf.xacro"/>
-  <!-- Include end-effectors -->
-  <xacro:include
-    filename="$(find blueprintlab_reachbravo7_manipulator_description)/urdf/end_effectors/jaws_macro.urdf.xacro"/>
-  <!-- Add manipulators-->
-  <xacro:reach_bravo7 prefix="$(arg bravo_namespace)" link6_lowlimit="0.0" link6_uplimit="3.14"/>
-  <!-- Attach manipulator to base -->
-  <joint name="girona1000_to_bravo" type="fixed">
-    <parent link="$(arg robot_namespace)/origin"/>
-    <child link="$(arg bravo_namespace)/base_link"/>
-    <origin rpy="${pi} 0.0 0.175" xyz="0.7322 0.1382 0.485"/>
-  </joint>
-  <xacro:reach_bravo7_jaws prefix="$(arg bravo_namespace)"/>
+  <xacro:if value="$(arg enable_arm)">
+    <!-- Include manipulators -->
+    <xacro:include
+      filename="$(find blueprintlab_reachbravo7_manipulator_description)/urdf/bravo7_macro.urdf.xacro"/>
+    <!-- Include end-effectors -->
+    <xacro:include
+      filename="$(find blueprintlab_reachbravo7_manipulator_description)/urdf/end_effectors/jaws_macro.urdf.xacro"/>
+    <!-- Add manipulators-->
+    <xacro:reach_bravo7 prefix="$(arg bravo_namespace)" link6_lowlimit="0.0" link6_uplimit="3.14"/>
+    <!-- Attach manipulator to base -->
+    <joint name="girona1000_to_bravo" type="fixed">
+      <parent link="$(arg robot_namespace)/origin"/>
+      <child link="$(arg bravo_namespace)/base_link"/>
+      <origin rpy="${pi} 0.0 0.175" xyz="0.7322 0.1382 0.485"/>
+    </joint>
+    <xacro:reach_bravo7_jaws prefix="$(arg bravo_namespace)"/>
+  </xacro:if>
   <link name="$(arg robot_namespace)/depth_cam_link"/>
   <joint name="$(arg robot_namespace)/depth_cam_joint" type="fixed">
@@ -33,10 +35,4 @@
     <child link="$(arg robot_namespace)/depth_cam_link"/>
     <origin rpy="1.309 0 1.57" xyz="0.7322 -0.1382 0.485"/>
-  </joint>
-  <link name="$(arg bravo_namespace)/gripper_camera"/>
-  <joint name="camera_joint" type="fixed">
-    <parent link="$(arg bravo_namespace)/jaws_base_link"/>
-    <child link="$(arg bravo_namespace)/gripper_camera"/>
-    <origin rpy="0 0 0" xyz="0 0 0.05"/>
   </joint>
   <link name="$(arg robot_namespace)/vlc_link"/>
